File: PCB/hairtag/hairtag.kicad_pcb (KiCad board)
At the start: 2 copper layers, 19 parts, among them J1 Flash, J2 BAT, U1 ESP32-C3FH4, U2 HT7533-1_C14289, X1 XL2EL89CPI-111YLC-40M

Commit message: asdf
Parts:
- removed C8: 1uF, lcsc:C0402
- J1: footprint Connector_PinHeader_2.54mm:PinHeader_1x06_P2.54mm_Vertical -> Connector_PinSocket_2.54mm:PinSocket_1x06_P2.54mm_Vertical
- moved L1 22.2 mm to (53.2, 54.8), turned to 90 degrees
- moved R2 21.8 mm to (57.5, 50.6), turned to 90 degrees
- moved R1 19.5 mm to (55.5, 58.9), turned to 90 degrees
- moved C9 19.1 mm to (57.5, 48.6), turned to -90 degrees
- moved C5 18.7 mm to (55.7, 50.2), turned to 180 degrees
- moved C10 18.3 mm to (58.8, 50.6), turned to -90 degrees
- moved AE1 17.4 mm to (50.8, 48.2), turned to 180 degrees
- moved C6 16.3 mm to (55.8, 51.5), turned to 180 degrees
- moved C3 16.2 mm to (52.8, 57.5)
- moved C2 16.1 mm to (52.8, 56.5)
- moved J1 15.9 mm to (51.8, 61.8), turned to 90 degrees
- moved X1 15.7 mm to (61.9, 49.4), turned to 180 degrees
- moved C1 14.4 mm to (54.5, 54.8), turned to 90 degrees
- moved C4 11.7 mm to (57.5, 58.9), turned to 90 degrees
- moved J2 11.6 mm to (50.0, 55.5)
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Connections:
- C1 pad 1: Net-(C1-Pad1) -> GND
- C1 pad 2: GND -> Net-(C1-Pad2)
- C2 pad 2: GND -> /VCC
- C3 pad 2: GND -> /VCC
- C4 pad 2: GND -> /VCC
- C5 pad 1: GND -> /VCC
- C6 pad 1: GND -> /VCC
- C7 pad 2: GND -> /VCC
- J1 pad 1: GND -> /VCC
- L1 pad 1: GND -> /VCC
- L1 pad 2: Net-(C1-Pad1) -> Net-(C1-Pad2)
- U1 pad 11: GND -> /VCC
- U1 pad 17: GND -> /VCC
- U1 pad 2: Net-(C1-Pad1) -> Net-(C1-Pad2)
- U1 pad 3: Net-(C1-Pad1) -> Net-(C1-Pad2)
- U1 pad 31: GND -> /VCC
- U1 pad 32: GND -> /VCC
- U2 pad 3: GND -> /VCC
Other:
- board outline added: 18 x 16.5 mm

Commit message: eee
Parts:
- moved J1 0.85 mm to (51.0, 61.6)
- moved C4 0.10 mm to (57.5, 58.8)
- moved R1 0.10 mm to (55.5, 58.8)
Other:
- board size 18 x 16.5 mm -> 20 x 20 mm
Changed lines of the file:
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@@
 	(footprint "lcsc:R0402"
 		(layer "F.Cu")
-		(at 55.5 58.93 90)
+		(at 55.5 58.83 90)
 		(property "Reference" "R1"
 			(at 0 -1 90)
@@
 	(footprint "Connector_PinSocket_2.54mm:PinSocket_1x06_P2.54mm_Vertical"
 		(layer "F.Cu")
-		(at 51.8 61.75 90)
+		(at 50.96 61.6 90)
 		(descr "Through hole straight socket strip, 1x06, 2.54mm pitch, single row (from Kicad 4.0.7), script generated")
 		(tags "Through hole socket strip THT 1x06 2.54mm single row")
 		(property "Reference" "J1"
-			(at 0 -2.77 90)
+			(at 0.5 -2.17 90)
 			(layer "F.SilkS")
 			(effects
@@
 		)
 		(property "Value" "Flash"
-			(at 0 15.47 90)
+			(at 1 15.33 90)
 			(layer "F.Fab")
 			(effects
@@
 	(footprint "lcsc:C0402"
 		(layer "F.Cu")
-		(at 57.5 58.92 90)
+		(at 57.5 58.82 90)
 		(property "Reference" "C4"
 			(at 0 -4 90)
@@
 		(layer "F.SilkS")
 	)
+	(gr_circle
+		(center 57.25 54.5)
+		(end 57.25 64.5)
+		(stroke
+			(width 0.05)
+			(type solid)
+		)
+		(fill no)
+		(layer "B.SilkS")
+	)
 	(gr_rect
-		(start 48.25 47)
-		(end 66.25 63.5)
+		(start 47.25 44.5)
+		(end 67.25 64.5)
+		(radius 5)
 		(stroke
 			(width 0.05)
-			(type default)
+			(type solid)
 		)
 		(fill no)

Commit message: ditch ldo
Parts:
- removed U2: HT7533-1_C14289, lcsc:SOT-89-3_L4.5-W2.5-P1.50-LS4.2-BR
Connections:
- J2 pad 1: /BAT+ -> /VCC

Commit message: cram
Parts:
- moved J1 1.45 mm to (50.0, 62.7), turned to 100 degrees
- moved X1 0.85 mm to (61.2, 49.9), turned to -90 degrees
Other:
- board size 20 x 20 mm -> 22 x 22 mm
Changed lines of the file:
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@@
 	(footprint "Connector_PinSocket_2.54mm:PinSocket_1x06_P2.54mm_Vertical"
 		(layer "F.Cu")
-		(at 50.96 61.6 90)
+		(at 49.997177 62.682133 100)
 		(descr "Through hole straight socket strip, 1x06, 2.54mm pitch, single row (from Kicad 4.0.7), script generated")
 		(tags "Through hole socket strip THT 1x06 2.54mm single row")
 		(property "Reference" "J1"
-			(at 0.5 -2.17 90)
+			(at 0.5 -2.17 100)
 			(layer "F.SilkS")
 			(effects
@@
 		)
 		(property "Value" "Flash"
-			(at 1 15.33 90)
+			(at 1 15.33 100)
 			(layer "F.Fab")
 			(effects
@@
 		)
 		(property "Datasheet" ""
-			(at 0 0 90)
+			(at 0 0 100)
 			(layer "F.Fab")
 			(hide yes)
@@
 		)
 		(property "Description" "Generic connector, single row, 01x06, script generated"
-			(at 0 0 90)
+			(at 0 0 100)
 			(layer "F.Fab")
 			(hide yes)
@@
 		)
 		(property "KiLib_Generator" "connector/pin_header_socket"
-			(at 0 0 90)
+			(at 0 0 100)
 			(layer "F.SilkS")
 			(hide yes)
@@
 		)
 		(fp_line
-			(start 1.33 1.27)
+			(start 1.329999 1.27)
 			(end 1.33 14.03)
 			(stroke
@@
 		(fp_line
 			(start -1.33 1.27)
-			(end 1.33 1.27)
+			(end 1.329999 1.27)
 			(stroke
 				(width 0.12)
@@
 		(fp_line
 			(start 1.77 14.47)
-			(end -1.77 14.47)
+			(end -1.77 14.469999)
 			(stroke
 				(width 0.05)
@@
 		)
 		(fp_line
-			(start -1.77 14.47)
+			(start -1.77 14.469999)
 			(end -1.77 -1.77)
 			(stroke
@@
 		(fp_line
 			(start 1.27 13.97)
-			(end -1.27 13.97)
+			(end -1.27 13.969999)
 			(stroke
 				(width 0.1)
@@
 		)
 		(fp_line
-			(start -1.27 13.97)
+			(start -1.27 13.969999)
 			(end -1.27 -1.27)
 			(stroke
@@
 		)
 		(fp_text user "${REFERENCE}"
-			(at 0 6.35 180)
+			(at 0 6.35 10)
 			(layer "F.Fab")
 			(effects
@@
 		)
 		(pad "1" thru_hole rect
-			(at 0 0 90)
+			(at 0 0 100)
 			(size 1.7 1.7)
 			(drill 1)
@@
 		)
 		(pad "2" thru_hole circle
-			(at 0 2.54 90)
+			(at 0 2.54 100)
 			(size 1.7 1.7)
 			(drill 1)
@@
 		)
 		(pad "3" thru_hole circle
-			(at 0 5.08 90)
+			(at 0 5.08 100)
 			(size 1.7 1.7)
 			(drill 1)
@@
 		)
 		(pad "4" thru_hole circle
-			(at 0 7.62 90)
+			(at 0 7.62 100)
 			(size 1.7 1.7)
 			(drill 1)
@@
 		)
 		(pad "5" thru_hole circle
-			(at 0 10.16 90)
+			(at -0.000001 10.16 100)
 			(size 1.7 1.7)
 			(drill 1)
@@
 		)
 		(pad "6" thru_hole circle
-			(at 0 12.7 90)
+			(at 0 12.7 100)
 			(size 1.7 1.7)
 			(drill 1)
@@
 	(footprint "lcsc:CRYSTAL-SMD_4P-L3.2-W2.5-BL"
 		(layer "F.Cu")
-		(at 61.9 49.35 180)
+		(at 61.25 49.9 -90)
 		(property "Reference" "X1"
-			(at 0 -4.85 0)
+			(at 0 -4.85 90)
 			(layer "F.SilkS")
 			(effects
@@
 		)
 		(property "Value" "XL2EL89CPI-111YLC-40M"
-			(at 0 4.85 0)
+			(at 0 4.85 90)
 			(layer "F.Fab")
 			(effects
@@
 		)
 		(property "Datasheet" "https://www.lcsc.com/datasheet/C5444549.pdf"
-			(at 0 0 0)
+			(at 0 0 90)
 			(layer "F.Fab")
 			(hide yes)
@@
 		)
 		(property "Description" ""
-			(at 0 0 0)
+			(at 0 0 90)
 			(layer "F.Fab")
 			(hide yes)
@@
 		)
 		(property "LCSC Part" "C5444549"
-			(at 0 0 0)
+			(at 0 0 90)
 			(layer "F.Fab")
 			(hide yes)
@@
 		)
 		(property "Manufacturer" "YXC(扬兴晶振)"
-			(at 0 0 180)
+			(at 0 0 270)
 			(unlocked yes)
 			(layer "F.Fab")
@@
 		)
 		(property "MPN" "XL2EL89CPI-111YLC-40M"
-			(at 0 0 180)
+			(at 0 0 270)
 			(unlocked yes)
 			(layer "F.Fab")
@@
 		(duplicate_pad_numbers_are_jumpers no)
 		(fp_line
-			(start 2.03 1.68)
-			(end -2.03 1.68)
+			(start -2.26 1.91)
+			(end -0.4 1.91)
 			(stroke
 				(width 0.15)
@@
 		)
 		(fp_line
-			(start 2.03 -1.68)
-			(end 2.03 1.68)
+			(start -2.03 1.68)
+			(end -2.03 -1.68)
 			(stroke
 				(width 0.15)
@@
 		)
 		(fp_line
-			(start -2.03 1.68)
-			(end -2.03 -1.68)
+			(start 2.03 1.68)
+			(end -2.03 1.68)
 			(stroke
 				(width 0.15)
@@
 		)
 		(fp_line
-			(start -2.03 -1.68)
-			(end 2.03 -1.68)
+			(start -2.26 0.25)
+			(end -2.26 1.91)
 			(stroke
 				(width 0.15)
@@
 		)
 		(fp_line
-			(start -2.26 1.91)
-			(end -0.4 1.91)
+			(start -2.03 -1.68)
+			(end 2.03 -1.68)
 			(stroke
 				(width 0.15)
@@
 		)
 		(fp_line
-			(start -2.26 0.25)
-			(end -2.26 1.91)
+			(start 2.03 -1.68)
+			(end 2.03 1.68)
 			(stroke
 				(width 0.15)
@@
 		)
 		(fp_line
-			(start 1.6 1.25)
-			(end -1.6 1.25)
+			(start -1.6 1.25)
+			(end -1.6 -1.25)
 			(stroke
 				(width 0.05)
@@
 		)
 		(fp_line
-			(start 1.6 -1.25)
-			(end 1.6 1.25)
+			(start 1.6 1.25)
+			(end -1.6 1.25)
 			(stroke
 				(width 0.05)
@@
 		)
 		(fp_line
-			(start -1.6 1.25)
-			(end -1.6 -1.25)
+			(start -1.6 -1.25)
+			(end 1.6 -1.25)
 			(stroke
 				(width 0.05)
@@
 		)
 		(fp_line
-			(start -1.6 -1.25)
-			(end 1.6 -1.25)
+			(start 1.6 -1.25)
+			(end 1.6 1.25)
 			(stroke
 				(width 0.05)
@@
 		)
 		(fp_text user "${REFERENCE}"
-			(at 0 0 0)
+			(at 0 0 90)
 			(layer "F.Fab")
 			(effects
@@
 		)
 		(pad "1" smd rect
-			(at -1.1 0.85 180)
+			(at -1.1 0.85 270)
 			(size 1.4 1.2)
 			(layers "F.Cu" "F.Mask" "F.Paste")
@@
 		)
 		(pad "2" smd rect
-			(at 1.1 0.85 180)
+			(at 1.1 0.85 270)
 			(size 1.4 1.2)
 			(layers "F.Cu" "F.Mask" "F.Paste")
@@
 		)
 		(pad "3" smd rect
-			(at 1.1 -0.85 180)
+			(at 1.1 -0.85 270)
 			(size 1.4 1.2)
 			(layers "F.Cu" "F.Mask" "F.Paste")
@@
 		)
 		(pad "4" smd rect
-			(at -1.1 -0.85 180)
+			(at -1.1 -0.85 270)
 			(size 1.4 1.2)
 			(layers "F.Cu" "F.Mask" "F.Paste")
@@
 	)
 	(gr_circle
-		(center 57.25 54.5)
-		(end 57.25 64.5)
-		(stroke
-			(width 0.05)
-			(type solid)
-		)
-		(fill no)
-		(layer "B.SilkS")
-	)
-	(gr_rect
-		(start 47.25 44.5)
-		(end 67.25 64.5)
-		(radius 5)
+		(center 55.1 55.4)
+		(end 66.1 55.4)
 		(stroke
 			(width 0.05)

Commit message: routing
Parts:
- moved R1 5.94 mm to (58.7, 63.8), turned to 0 degrees
- moved X1 0.71 mm to (61.1, 49.2)
- renumbered J2 to BAT+, J1 to Flash
Routing:
- net /VCC: track 0.00 -> 35.7 mm, vias 0 -> 4
- net Net-(U1-U0TXD): track 0.00 -> 19.9 mm
- net GND: track 0.00 -> 19.8 mm, vias 0 -> 8
- net /TXD: track 0.00 -> 18.8 mm
- net /CHIP_EN: track 0.00 -> 8.51 mm, vias 0 -> 2
- net /XTAL_N: track 0.00 -> 7.42 mm
- net /LNA_IN: track 0.00 -> 6.42 mm
- net /CTS: track 0.00 -> 5.48 mm, vias 0 -> 2
- net Net-(C9-Pad2): track 0.00 -> 4.33 mm
- net Net-(C1-Pad2): track 0.00 -> 3.01 mm
- net /RXD: track 0.00 -> 2.79 mm
- net /XTAL_P: track 0.00 -> 1.41 mm
- added copper zone on B.Cu, net GND
- added copper zone on F.Cu, net GND
Other:
- board size 22 x 22 mm -> 23 x 23 mm
- board text added: "@jblitzar"

Commit message: misc stuff
Parts:
- moved R1 1.10 mm to (59.8, 63.8)
- renumbered AE1 to 2450AT18A100E, X1 to YSX321SL, U1 to esp32c3fh4
Routing:
- net /VCC: track 35.7 -> 54.3 mm
- net Net-(U1-U0TXD): track 19.9 -> 18.8 mm
- net /RXD: track 2.79 -> 3.88 mm
Other:
- board text added: "CTS"
- board text added: "GND"
- board text added: "RTS"
- board text added: "RXD"
- board text added: "TXD"
- board text added: "VCC"
- board text added: "by @jblitzar"
- board text added: "hairtag"
- board text removed: "@jblitzar"

Commit message: readme stuff
Parts:
- removed BAT+: BAT, Connector_PinHeader_2.54mm:PinHeader_1x02_P2.54mm_Vertical
- removed Flash: Flash, Connector_PinSocket_2.54mm:PinSocket_1x06_P2.54mm_Vertical
- added J1: Flash, Connector_PinSocket_2.54mm:PinSocket_1x06_P2.54mm_Vertical, F.Cu at (48.8, 61.6)
- added J2: BAT, cr2032_holder:Untitled, F.Cu at (55.2, 58.6)
- renumbered 2450AT18A100E to AE1, esp32c3fh4 to U1, YSX321SL to X1
Routing:
- net /CTS: track 5.61 -> 7.16 mm
- net /TXD: track 19.1 -> 20.1 mm
- net /VCC: track 54.3 -> 53.6 mm
- net GND: vias 8 -> 9
Other:
- board size 23 x 23 mm -> 24 x 24 mm
- board text removed: "CTS"
- board text removed: "GND"
- board text removed: "RTS"
- board text removed: "RXD"
- board text removed: "TXD"
- board text removed: "VCC"
