File: PCB/hairtag/hairtag.kicad_sch (KiCad schematic)
At the start: 19 parts, among them J1 Flash, J2 BAT, U1 ESP32-C3FH4, U2 HT7533-1_C14289, X1 XL2EL89CPI-111YLC-40M

Commit message: asdf
Parts:
- removed C8: 1uF, lcsc:C0402, symbol lcsc:CL05A105KO5NNNC
- J1: footprint Connector_PinHeader_2.54mm:PinHeader_1x06_P2.54mm_Vertical -> Connector_PinSocket_2.54mm:PinSocket_1x06_P2.54mm_Vertical
Connections:
- net GND: now also C1.1; no longer C1.2, C2.2, C3.2, C4.2, C5.1, C6.1, C7.2, J1.1 (Pin_1), L1.1, U1.11 (VDD3P3_RTC), U1.17 (VDD3P3_CPU), U1.31 (VDDA), U1.32 (VDDA), U2.3 (Vout)
- net at L1.2, U1.2 (VDD3P3), U1.3 (VDD3P3): now also C1.2; no longer C1.1
- new net VCC: C2.2, C3.2, C4.2, C5.1, C6.1, C7.2, J1.1 (Pin_1), L1.1, U1.11 (VDD3P3_RTC), U1.17 (VDD3P3_CPU), U1.31 (VDDA), U1.32 (VDDA), U2.3 (Vout)
Other:
- moved on the sheet: C1, C6

Commit message: ditch ldo
Parts:
- removed U2: HT7533-1_C14289, lcsc:SOT-89-3_L4.5-W2.5-P1.50-LS4.2-BR, symbol lcsc:HT7533-1_C14289
Connections:
- net BAT+ is gone; now on net VCC: J2.1 (Pin_1)
Changed lines of the file:
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@@
-		)
-	)
-	(label "BAT+"
-		(at 217.17 104.14 180)
-		(effects
-			(font
-				(size 1.27 1.27)
-			)
-			(justify right bottom)
 		)
 	)
@@
 		)
 	)
-	(label "BAT+"
+	(label "VCC"
 		(at 266.7 104.14 180)
 		(effects
@@
 			)
 			(justify right bottom)
-		)
-	)
-	(label "VCC"
-		(at 237.49 99.06 0)
-		(effects
-			(font
-				(size 1.27 1.27)
-			)
-			(justify left bottom)
 		)
 	)
@@
 	(symbol
 		(lib_id "power:GND")
-		(at 237.49 109.22 0)
-		(unit 1)
-		(body_style 1)
-		(exclude_from_sim no)
-		(in_bom yes)
-		(on_board yes)
-		(in_pos_files yes)
-		(dnp no)
-		(fields_autoplaced yes)
-		(property "Reference" "#PWR02"
-			(at 237.49 115.57 0)
-			(hide yes)
-			(show_name no)
-			(do_not_autoplace no)
-			(effects
-				(font
-					(size 1.27 1.27)
-				)
-			)
-		)
-		(property "Value" "GND"
-			(at 237.49 114.3 0)
-			(show_name no)
-			(do_not_autoplace no)
-			(effects
-				(font
-					(size 1.27 1.27)
-				)
-			)
-		)
-		(property "Footprint" ""
-			(at 237.49 109.22 0)
-			(hide yes)
-			(show_name no)
-			(do_not_autoplace no)
-			(effects
-				(font
-					(size 1.27 1.27)
-				)
-			)
-		)
-		(property "Datasheet" ""
-			(at 237.49 109.22 0)
-			(hide yes)
-			(show_name no)
-			(do_not_autoplace no)
-			(effects
-				(font
-					(size 1.27 1.27)
-				)
-			)
-		)
-		(property "Description" "Power symbol creates a global label with name \"GND\" , ground"
-			(at 237.49 109.22 0)
-			(hide yes)
-			(show_name no)
-			(do_not_autoplace no)
-			(effects
-				(font
-					(size 1.27 1.27)
-				)
-			)
-		)
-		(pin "1"
-		)
-		(instances
-			(project "hairtag"
-				(path "/aa294e8c-6ec0-4a40-9993-950bbf2ffeff"
-					(reference "#PWR02")
-					(unit 1)
-				)
-			)
-		)
-	)
-	(symbol
-		(lib_id "power:GND")
 		(at 234.95 35.56 0)
 		(unit 1)
@@
 					(unit 1)
 				)
-			)
-		)
-	)
-	(symbol
-		(lib_id "lcsc:HT7533-1_C14289")
-		(at 227.33 104.14 0)
-		(unit 1)
-		(body_style 1)
-		(exclude_from_sim no)
-		(in_bom yes)
-		(on_board yes)
-		(in_pos_files yes)
-		(dnp no)
-		(fields_autoplaced yes)
-		(property "Reference" "U2"
-			(at 227.33 91.44 0)
-			(show_name no)
-			(do_not_autoplace no)
-			(effects
-				(font
-					(size 1.27 1.27)
-				)
-			)
-		)
-		(property "Value" "HT7533-1_C14289"
-			(at 227.33 93.98 0)
-			(show_name no)
-			(do_not_autoplace no)
-			(effects
-				(font
-					(size 1.27 1.27)
-				)
-			)
-		)
-		(property "Footprint" "lcsc:SOT-89-3_L4.5-W2.5-P1.50-LS4.2-BR"
-			(at 227.33 116.84 0)
-			(hide yes)
-			(show_name no)
-			(do_not_autoplace no)
-			(effects
-				(font
-					(size 1.27 1.27)
-				)
-			)
-		)
-		(property "Datasheet" "https://lcsc.com/product-detail/Low-Dropout-Regulators-LDO_HT7533-1_C14289.html"
-			(at 227.33 119.38 0)
-			(hide yes)
-			(show_name no)
-			(do_not_autoplace no)
-			(effects
-				(font
-					(size 1.27 1.27)
-				)
-			)
-		)
-		(property "Description" ""
-			(at 227.33 104.14 0)
-			(hide yes)
-			(show_name no)
-			(do_not_autoplace no)
-			(effects
-				(font
-					(size 1.27 1.27)
-				)
-			)
-		)
-		(property "Manufacturer" "HOLTEK(合泰/盛群)"
-			(at 227.33 121.92 0)
-			(hide yes)
-			(show_name no)
-			(do_not_autoplace no)
-			(effects
-				(font
-					(size 1.27 1.27)
-				)
-			)
-		)
-		(property "MPN" "HT7533-1"
-			(at 227.33 124.46 0)
-			(hide yes)
-			(show_name no)
-			(do_not_autoplace no)
-			(effects
-				(font
-					(size 1.27 1.27)
-				)
-			)
-		)
-		(property "LCSC Part" "C14289"
-			(at 227.33 127 0)
-			(hide yes)
-			(show_name no)
-			(do_not_autoplace no)
-			(effects
-				(font
-					(size 1.27 1.27)
-				)
-			)
-		)
-		(pin "2"
-		)
-		(pin "1"
-		)
-		(pin "3"
-		)
-		(instances
-			(project "hairtag"
-				(path "/aa294e8c-6ec0-4a40-9993-950bbf2ffeff"
-					(reference "U2")
-					(unit 1)
-				)

Commit message: misc stuff
Parts:
- C1, C5: LCSC Part C29266 -> C52923; MPN CL05A105KO5NNNC -> CL05A105KA5NQNC
- C10, C9: LCSC Part C86285 -> C1548; MPN CL05C150JB5NNNC -> 0402CG150J500NT
- C2, C4, C7: LCSC Part C60474 -> C1525; MPN CC0402KRX7R7BB104 -> CL05B104KO5NNNC
- C3: symbol lcsc:CL05A106MP5NUNC_C315248 -> lcsc:CL05A106MP5NUNC_C15525; LCSC Part C315248 -> C15525; MPN CL05A106MP5NUNC -> CL05A106MQ5NUNC
Changed lines of the file:
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@@
 	)
 	(symbol
-		(lib_id "lcsc:CL05A106MP5NUNC_C315248")
+		(lib_id "lcsc:CL05A106MP5NUNC_C15525")
 		(at 66.04 77.47 90)
 		(unit 1)
@@
 			)
 		)
-		(property "MPN" "CL05A106MP5NUNC"
+		(property "MPN" "CL05A106MQ5NUNC"
 			(at 81.28 77.47 0)
 			(hide yes)
@@
 			)
 		)
-		(property "LCSC Part" "C315248"
+		(property "LCSC Part" "C15525"
 			(at 83.82 77.47 0)
 			(hide yes)
@@
 			)
 		)
-		(property "Datasheet" "https://lcsc.com/product-detail/Others_Samsung-Electro-Mechanics_CL05C150JB5NNNC_Samsung-Electro-Mechanics-CL05C150JB5NNNC_C86285.html"
+		(property "Datasheet" "https://lcsc.com/product-detail/Others_Samsung-Electro-Mechanics_CL05C150JB5NNNC_Samsung-Electro-Mechanics-CL05C150JB5NNNC_C1548.html"
 			(at 196.85 59.69 0)
 			(hide yes)
@@
 			)
 		)
-		(property "MPN" "CL05C150JB5NNNC"
+		(property "MPN" "0402CG150J500NT"
 			(at 196.85 64.77 0)
 			(hide yes)
@@
 			)
 		)
-		(property "LCSC Part" "C86285"
+		(property "LCSC Part" "C1548"
 			(at 196.85 67.31 0)
 			(hide yes)
@@
 			)
 		)
-		(property "Datasheet" "https://lcsc.com/product-detail/Multilayer-Ceramic-Capacitors-MLCC-SMD-SMT_100nF-104-10-16V_C60474.html"
+		(property "Datasheet" "https://lcsc.com/product-detail/Multilayer-Ceramic-Capacitors-MLCC-SMD-SMT_100nF-104-10-16V_C1525.html"
 			(at 157.48 113.03 0)
 			(hide yes)
@@
 			)
 		)
-		(property "MPN" "CC0402KRX7R7BB104"
+		(property "MPN" "CL05B104KO5NNNC"
 			(at 162.56 113.03 0)
 			(hide yes)
@@
 			)
 		)
-		(property "LCSC Part" "C60474"
+		(property "LCSC Part" "C1525"
 			(at 165.1 113.03 0)
 			(hide yes)
@@
 			)
 		)
-		(property "Datasheet" "https://lcsc.com/product-detail/Multilayer-Ceramic-Capacitors-MLCC-SMD-SMT_100nF-104-10-16V_C60474.html"
+		(property "Datasheet" "https://lcsc.com/product-detail/Multilayer-Ceramic-Capacitors-MLCC-SMD-SMT_100nF-104-10-16V_C1525.html"
 			(at 95.25 100.33 0)
 			(hide yes)
@@
 			)
 		)
-		(property "MPN" "CC0402KRX7R7BB104"
+		(property "MPN" "CL05B104KO5NNNC"
 			(at 100.33 100.33 0)
 			(hide yes)
@@
 			)
 		)
-		(property "LCSC Part" "C60474"
+		(property "LCSC Part" "C1525"
 			(at 102.87 100.33 0)
 			(hide yes)
@@
 			)
 		)
-		(property "Datasheet" "https://lcsc.com/product-detail/Multilayer-Ceramic-Capacitors-MLCC-SMD-SMT_100nF-104-10-16V_C60474.html"
+		(property "Datasheet" "https://lcsc.com/product-detail/Multilayer-Ceramic-Capacitors-MLCC-SMD-SMT_100nF-104-10-16V_C1525.html"
 			(at 83.82 77.47 0)
 			(hide yes)
@@
 			)
 		)
-		(property "MPN" "CC0402KRX7R7BB104"
+		(property "MPN" "CL05B104KO5NNNC"
 			(at 88.9 77.47 0)
 			(hide yes)
@@
 			)
 		)
-		(property "LCSC Part" "C60474"
+		(property "LCSC Part" "C1525"
 			(at 91.44 77.47 0)
 			(hide yes)
@@
 			)
 		)
-		(property "Datasheet" "https://lcsc.com/product-detail/Multilayer-Ceramic-Capacitors-MLCC-SMD-SMT_SAMSUNG_CL05A105KO5NNNC_1uF-105-10-16V_C29266.html"
+		(property "Datasheet" "https://lcsc.com/product-detail/Multilayer-Ceramic-Capacitors-MLCC-SMD-SMT_SAMSUNG_CL05A105KO5NNNC_1uF-105-10-16V_C52923.html"
 			(at 161.29 62.23 0)
 			(hide yes)
@@
 			)
 		)
-		(property "MPN" "CL05A105KO5NNNC"
+		(property "MPN" "CL05A105KA5NQNC"
 			(at 156.21 62.23 0)
 			(hide yes)
@@
 			)
 		)
-		(property "LCSC Part" "C29266"
+		(property "LCSC Part" "C52923"
 			(at 153.67 62.23 0)
 			(hide yes)
@@
 			)
 		)
-		(property "Datasheet" "https://lcsc.com/product-detail/Others_Samsung-Electro-Mechanics_CL05C150JB5NNNC_Samsung-Electro-Mechanics-CL05C150JB5NNNC_C86285.html"
+		(property "Datasheet" "https://lcsc.com/product-detail/Others_Samsung-Electro-Mechanics_CL05C150JB5NNNC_Samsung-Electro-Mechanics-CL05C150JB5NNNC_C1548.html"
 			(at 196.85 41.91 0)
 			(hide yes)
@@
 			)
 		)
-		(property "MPN" "CL05C150JB5NNNC"
+		(property "MPN" "0402CG150J500NT"
 			(at 196.85 46.99 0)
 			(hide yes)
@@
 			)
 		)
-		(property "LCSC Part" "C86285"
+		(property "LCSC Part" "C1548"
 			(at 196.85 49.53 0)
 			(hide yes)
@@
 			)
 		)
-		(property "Datasheet" "https://lcsc.com/product-detail/Multilayer-Ceramic-Capacitors-MLCC-SMD-SMT_SAMSUNG_CL05A105KO5NNNC_1uF-105-10-16V_C29266.html"
+		(property "Datasheet" "https://lcsc.com/product-detail/Multilayer-Ceramic-Capacitors-MLCC-SMD-SMT_SAMSUNG_CL05A105KO5NNNC_1uF-105-10-16V_C52923.html"
 			(at 93.98 76.2 0)
 			(hide yes)
@@
 			)
 		)
-		(property "MPN" "CL05A105KO5NNNC"
+		(property "MPN" "CL05A105KA5NQNC"
 			(at 99.06 76.2 0)
 			(hide yes)
@@
 			)
 		)
-		(property "LCSC Part" "C29266"
+		(property "LCSC Part" "C52923"
 			(at 101.6 76.2 0)
 			(hide yes)

Commit message: readme stuff
Parts:
- J2: footprint Connector_PinHeader_2.54mm:PinHeader_1x02_P2.54mm_Vertical -> cr2032_holder:Untitled
Changed lines of the file:
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@@
 			)
 		)
-		(property "Footprint" "Connector_PinHeader_2.54mm:PinHeader_1x02_P2.54mm_Vertical"
+		(property "Footprint" "cr2032_holder:Untitled"
 			(at 271.78 104.14 0)
 			(hide yes)

Commit message: stuff
Connections:
- net GND: now also J2.1 (Pin_1); no longer J2.2 (Pin_2)
- net VCC: now also J2.2 (Pin_2); no longer J2.1 (Pin_1)
- net CTS renamed DTR
Changed lines of the file:
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@@
-		)
-	)
-	(label "VCC"
-		(at 266.7 104.14 180)
-		(effects
-			(font
-				(size 1.27 1.27)
-			)
-			(justify right bottom)
 		)
 	)
@@
 		)
 	)
-	(label "CTS"
+	(label "DTR"
 		(at 195.58 140.97 0)
 		(effects
@@
 		)
 	)
-	(label "CTS"
+	(label "DTR"
 		(at 220.98 139.7 180)
 		(effects
@@
 			)
 			(justify left bottom)
+		)
+	)
+	(label "VCC"
+		(at 266.7 106.68 180)
+		(effects
+			(font
+				(size 1.27 1.27)
+			)
+			(justify right bottom)
 		)
 	)
@@
 	)
 	(symbol
+		(lib_id "power:GND")
+		(at 266.7 104.14 270)
+		(unit 1)
+		(body_style 1)
+		(exclude_from_sim no)
+		(in_bom yes)
+		(on_board yes)
+		(in_pos_files yes)
+		(dnp no)
+		(fields_autoplaced yes)
+		(property "Reference" "#PWR03"
+			(at 260.35 104.14 0)
+			(hide yes)
+			(show_name no)
+			(do_not_autoplace no)
+			(effects
+				(font
+					(size 1.27 1.27)
+				)
+			)
+		)
+		(property "Value" "GND"
+			(at 262.89 104.1399 90)
+			(show_name no)
+			(do_not_autoplace no)
+			(effects
+				(font
+					(size 1.27 1.27)
+				)
+				(justify right)
+			)
+		)
+		(property "Footprint" ""
+			(at 266.7 104.14 0)
+			(hide yes)
+			(show_name no)
+			(do_not_autoplace no)
+			(effects
+				(font
+					(size 1.27 1.27)
+				)
+			)
+		)
+		(property "Datasheet" ""
+			(at 266.7 104.14 0)
+			(hide yes)
+			(show_name no)
+			(do_not_autoplace no)
+			(effects
+				(font
+					(size 1.27 1.27)
+				)
+			)
+		)
+		(property "Description" "Power symbol creates a global label with name \"GND\" , ground"
+			(at 266.7 104.14 0)
+			(hide yes)
+			(show_name no)
+			(do_not_autoplace no)
+			(effects
+				(font
+					(size 1.27 1.27)
+				)
+			)
+		)
+		(pin "1"
+		)
+		(instances
+			(project "hairtag"
+				(path "/aa294e8c-6ec0-4a40-9993-950bbf2ffeff"
+					(reference "#PWR03")
+					(unit 1)
+				)
+			)
+		)
+	)
+	(symbol
 		(lib_id "lcsc:CC0402KRX7R7BB104")
 		(at 147.32 113.03 90)
@@
 					(unit 1)
 				)
-			)
-		)
-	)
-	(symbol
-		(lib_id "power:GND")
-		(at 266.7 106.68 0)
-		(unit 1)
-		(body_style 1)
-		(exclude_from_sim no)
-		(in_bom yes)
-		(on_board yes)
-		(in_pos_files yes)
-		(dnp no)
-		(fields_autoplaced yes)
-		(property "Reference" "#PWR03"
-			(at 266.7 113.03 0)
-			(hide yes)
-			(show_name no)
-			(do_not_autoplace no)
-			(effects
-				(font
-					(size 1.27 1.27)
-				)
-			)
-		)
-		(property "Value" "GND"
-			(at 266.7 111.76 0)
-			(show_name no)
-			(do_not_autoplace no)
-			(effects
-				(font
-					(size 1.27 1.27)
-				)
-			)
-		)
-		(property "Footprint" ""
-			(at 266.7 106.68 0)
-			(hide yes)
-			(show_name no)
-			(do_not_autoplace no)
-			(effects
-				(font
-					(size 1.27 1.27)
-				)
-			)
-		)
-		(property "Datasheet" ""
-			(at 266.7 106.68 0)
-			(hide yes)
-			(show_name no)
-			(do_not_autoplace no)
-			(effects
-				(font
-					(size 1.27 1.27)
-				)
-			)
-		)
-		(property "Description" "Power symbol creates a global label with name \"GND\" , ground"
-			(at 266.7 106.68 0)
-			(hide yes)
-			(show_name no)
-			(do_not_autoplace no)
-			(effects
-				(font
-					(size 1.27 1.27)
-				)
-			)
-		)
-		(pin "1"
-		)
-		(instances
-			(project "hairtag"
-				(path "/aa294e8c-6ec0-4a40-9993-950bbf2ffeff"
-					(reference "#PWR03")
-					(unit 1)
-				)

Commit message: add LED
Parts:
- added LED1: FC-1608YXK-585F08, lcsc:LED0603-RD, symbol lcsc:FC-1608YXK-585F08
- added R3: 0402WGF3300TCE, lcsc:R0402, symbol lcsc:0402WGF3300TCE
Connections:
- net GND: now also LED1.1 (K)
- net GPIO10: now also R3.2
- new net: LED1.2 (A), R3.1

Commit message: tweaks
Parts:
- removed R2: 24Ω, lcsc:R0402, symbol lcsc:0402WGF240JTCE
- added C11: 100uF, lcsc:C1206, symbol lcsc:CL31A107MQHNNNE
- added C8: 1uF, lcsc:C0402, symbol lcsc:CL05A105KO5NNNC
- added L2: 15nH, lcsc:L0402, symbol lcsc:SDCL1005C15NJTDF
- added R2, R7: 22, lcsc:R0402, symbol lcsc:0402WGF220JTCE
- added R4, R5, R6: 10k, lcsc:R0402, symbol lcsc:0402WGF1002TCE
- added USB1: USB, Connector_PinSocket_2.54mm:PinSocket_1x02_P2.54mm_Vertical, symbol Connector:Conn_01x02_Socket
- L1: value (none) -> 2nF
Connections:
- net CHIP_EN: now also C8.2, R4.2
- net GND: now also C11.1, C8.1
- net GPIO18: now also R7.1
- net GPIO19: now also R2.1
- net GPIO2: now also R6.1
- net GPIO8: now also R5.1
- net VCC: now also C11.2, R4.1, R5.2, R6.2
- net XTAL_P: now also L2.1
- net at C9.2, X1.1: now also L2.2
- new net: R7.2, USB1.2 (Pin_2)
- new net: R2.2, USB1.1 (Pin_1)

Commit message: ordered it!
Parts:
- J1, J2: now not fitted; now left out of the parts list
Changed lines of the file:
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@@
 		(body_style 1)
 		(exclude_from_sim no)
-		(in_bom yes)
-		(on_board yes)
-		(in_pos_files yes)
-		(dnp no)
+		(in_bom no)
+		(on_board yes)
+		(in_pos_files yes)
+		(dnp yes)
 		(fields_autoplaced yes)
 		(property "Reference" "J2"
@@
 		(body_style 1)
 		(exclude_from_sim no)
-		(in_bom yes)
-		(on_board yes)
-		(in_pos_files yes)
-		(dnp no)
+		(in_bom no)
+		(on_board yes)
+		(in_pos_files yes)
+		(dnp yes)
 		(fields_autoplaced yes)
 		(property "Reference" "J1"
