File: PCB/hairtag/hairtag.kicad_sch (KiCad schematic)
At the start: 27 parts, among them J1 Flash, J2 BAT, U1 ESP32-C3FH4, X1 XL2EL89CPI-111YLC-40M

Commit message: OMG OMG OMG
Parts:
- added C12: 1pF, easyeda2kicad:C0402, symbol lcsc:CC0402BRNPO9BN1R0
- added L3: 2.7nH, easyeda2kicad:L0402, symbol lcsc:LQG15HS2N7S02D
- added L4: 3.9nH, easyeda2kicad:IND-SMD_L1.0-W0.5-2, symbol lcsc:LQW15AN3N9B00D
Connections:
- net GND: now also L3.1
- net LNA_IN: now also C12.1; no longer AE1.1 (ANT)
- new net: AE1.1 (ANT), L4.1
- new net: C12.2, L3.2, L4.2
