File: PCB/hairtag/hairtag.kicad_sch (KiCad schematic)
At the start: 30 parts, among them J1 Flash, J2 BAT, U1 ESP32-C3FH4, X1 XL2EL89CPI-111YLC-40M

Commit message: bom fix
Parts:
- C12: LCSC Part C309455 -> C1550; MPN CC0402BRNPO9BN1R0 -> 0402CG1R0C500NT; Manufacturer YAGEO(国巨) -> Guangdong Fenghua(风华高科)
- L1: value 2nF -> 2nH
- L3: LCSC Part C77108 -> C27123; MPN LQG15HS2N7S02D -> SDCL1005C2N7STDF; Manufacturer muRata(村田) -> Sunlord(顺络)
- LED1: LCSC Part C89811 -> C2286; MPN NCD0603Y2 -> KT-0603R; Manufacturer 国星光电 -> Hubei KENTO Elec
- USB1: now not fitted; now left out of the parts list
Changed lines of the file:
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@@
 			)
 		)
-		(property "Value" "2nF"
+		(property "Value" "2nH"
 			(at 78.71 68.58 0)
 			(show_name no)
@@
 			)
 		)
-		(property "Datasheet" "https://lcsc.com/product-detail/_FC-1608YXK-585F08_C89811.html"
+		(property "Datasheet" "https://www.lcsc.com/product-detail/C2286.html"
 			(at 57.15 140.97 0)
 			(hide yes)
@@
 			)
 		)
-		(property "Manufacturer" "国星光电"
+		(property "Manufacturer" "Hubei KENTO Elec"
 			(at 57.15 143.51 0)
 			(hide yes)
@@
 			)
 		)
-		(property "MPN" "NCD0603Y2"
+		(property "MPN" "KT-0603R"
 			(at 57.15 146.05 0)
 			(hide yes)
@@
 			)
 		)
-		(property "LCSC Part" "C89811"
+		(property "LCSC Part" "C2286"
 			(at 57.15 148.59 0)
 			(hide yes)
@@
 			)
 		)
-		(property "Datasheet" "https://lcsc.com/product-detail/HF-Inductors_muRata_LQG15HS2N7S02D_2-7nH-0-3nH_C77108.html"
+		(property "Datasheet" "https://www.lcsc.com/product-detail/C27123.html"
 			(at 265.43 82.55 0)
 			(hide yes)
@@
 			)
 		)
-		(property "Manufacturer" "muRata(村田)"
+		(property "Manufacturer" "Sunlord(顺络)"
 			(at 267.97 82.55 0)
 			(hide yes)
@@
 			)
 		)
-		(property "MPN" "LQG15HS2N7S02D"
+		(property "MPN" "SDCL1005C2N7STDF"
 			(at 270.51 82.55 0)
 			(hide yes)
@@
 			)
 		)
-		(property "LCSC Part" "C77108"
+		(property "LCSC Part" "C27123"
 			(at 273.05 82.55 0)
 			(hide yes)
@@
 			)
 		)
-		(property "Datasheet" "https://lcsc.com/product-detail/Others_YAGEO-CC0402BRNPO9BN1R0_C309455.html"
+		(property "Datasheet" "https://www.lcsc.com/product-detail/C1550.html"
 			(at 275.59 77.47 0)
 			(hide yes)
@@
 			)
 		)
-		(property "Manufacturer" "YAGEO(国巨)"
+		(property "Manufacturer" "Guangdong Fenghua(风华高科)"
 			(at 278.13 77.47 0)
 			(hide yes)
@@
 			)
 		)
-		(property "MPN" "CC0402BRNPO9BN1R0"
+		(property "MPN" "0402CG1R0C500NT"
 			(at 280.67 77.47 0)
 			(hide yes)
@@
 			)
 		)
-		(property "LCSC Part" "C309455"
+		(property "LCSC Part" "C1550"
 			(at 283.21 77.47 0)
 			(hide yes)
@@
 		(body_style 1)
 		(exclude_from_sim no)
-		(in_bom yes)
+		(in_bom no)
 		(on_board yes)
 		(in_pos_files yes)
-		(dnp no)
+		(dnp yes)
 		(fields_autoplaced yes)
 		(property "Reference" "USB1"
